File: PDP-8-Serial.kicad_sch (KiCad schematic)
At the start: 57 parts, among them J1 FlipChip_01x18, J2 Screw_Terminal_01x06, J3 DE9_Socket_MountingHoles, Q1 2N3906, U1 L78L05_TO92, U2 74HCT14, U3 MAX232

Commit message: Improved Tx side level translation
Parts:
- removed R13: 2k2, Resistor_THT:R_Axial_DIN0207_L6.3mm_D2.5mm_P10.16mm_Horizontal, symbol Device:R
- added D4, D5: 1N914, Diode_THT:D_DO-35_SOD27_P7.62mm_Horizontal, symbol Diode:1N914
- added Q1, Q2: 2N3904, Package_TO_SOT_THT:TO-92_Inline, symbol Transistor_BJT:2N3904
- added R12: 330k, Resistor_THT:R_Axial_DIN0207_L6.3mm_D2.5mm_P10.16mm_Horizontal, symbol Device:R
- R10: renamed from R4; value 33k -> 330k
- R3: renamed from R2; value 1K -> 1k
- R4: renamed from R11; value 2k2 -> 1k
- R5: renamed from R12; value 2k2 -> 1k
- R6: value 7k5 -> 1k
- R7: value 33k -> 47k
- R9: value 7k5 -> 47k
- renumbered C2 to C1, C13 to C10, C6 to C12, C9 to C13, C3 to C2, C5 to C3, C12 to C4, C10 to C5, C7 to C6, C4 to C7, C1 to C8, C8 to C9, D5 to D1, D7 to D10, D6 to D11, D4 to D2, D1 to D6, D10 to D7, D9 to D8, D8 to D9, J2 to J1, J3 to J2, J1 to J3, LK3 to LK1, LK1 to LK2, LK2 to LK3, Q1 to Q3, R10 to R1, R5 to R11, R14 to R13, R15 to R14, R16 to R15, R3 to R2, TP4 to TP1, TP1 to TP2, TP5 to TP3, TP6 to TP4, TP7 to TP5, TP2 to TP6, TP3 to TP7, U3 to U1, U1 to U3
Connections:
- net +5V: now also R5.2, R6.2, R9.1, R12.1; no longer R5.1
- net -15V: no longer R6.2, R9.2
- net GND: now also D4.2 (A), D5.2 (A), Q1.1 (E), Q2.1 (E)
- net at JP3.2 (C), U1.10 (T2IN): now also D3.1 (K)
- net at JP2.2 (C), U1.11 (T1IN): now also D2.1 (K)
- net at U1.12 (R1OUT), U2.1: no longer U2.13
- net at JP3.3 (B), U2.10, U2.9: no longer D3.1 (K)
- net at JP2.3 (B), U2.4, U2.5: no longer D2.1 (K)
- net at D2.2 (A): now also R5.1; no longer R5.2
- net at D1.1 (K), U2.12: now also R13.1
- net at D3.2 (A): now also R6.1
- net at U2.2: now also U2.13; no longer R13.1
- new net: Q1.3 (C), R9.2, U2.11
- new net: Q2.3 (C), R7.2, U2.3
- new net: D5.1 (K), Q1.2 (B), R12.2, R8.2
- new net: LK3.1 (Pin_1), R11.1
- new net: D4.1 (K), Q2.2 (B), R10.2, R11.2
- new net: LK1.1 (Pin_1), R8.1
Other:
- moved on the sheet: C13, D1, D10, D11, D2, D7, D8, D9, JP2, Q3, R10, R11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
