File: PDP-8-Serial.kicad_pcb (KiCad board)
At the start: 2 copper layers, 125.7 x 62.2 mm, 57 parts, among them J1 FlipChip_01x18, J2 Screw_Terminal_01x06, J3 DE9_Socket_MountingHoles, Q1 2N3906, U1 L78L05_TO92, U2 74HCT14, U3 MAX232

Commit message: Improved Tx side level translation
Parts:
- removed the R6 at (147.4, 118.5)
- added D4: 1N914, Diode_THT:D_DO-35_SOD27_P7.62mm_Horizontal, F.Cu at (131.3, 94.6)
- added D5: 1N914, Diode_THT:D_DO-35_SOD27_P7.62mm_Horizontal, F.Cu at (131.3, 97.4)
- added Q1: 2N3904, Package_TO_SOT_THT:TO-92_Inline, F.Cu at (135.8, 94.7)
- added Q2: 2N3904, Package_TO_SOT_THT:TO-92_Inline, F.Cu at (142.8, 94.7)
- added R7: 47k, Resistor_THT:R_Axial_DIN0207_L6.3mm_D2.5mm_P10.16mm_Horizontal, F.Cu at (157.6, 96.4)
- R10: renamed from R4; value 33k -> 330k
- R12: renamed from R8; value 100k -> 330k
- R3: renamed from R2; value 1K -> 1k
- R4: renamed from R11; value 2k2 -> 1k
- R5: renamed from R12; value 2k2 -> 1k
- R6: renamed from R13; value 2k2 -> 1k
- R8: renamed from R9; value 7k5 -> 100k
- R9: renamed from R7; value 33k -> 47k
- moved TP1 21.7 mm to (147.6, 74.5)
- moved R13 15.8 mm to (147.4, 115.3)
- moved R8 15.7 mm to (157.6, 99.6)
- moved R12 10.2 mm to (157.6, 112.2), turned to 180 degrees
- moved R5 10.2 mm to (108.2, 107.3), turned to -90 degrees
- moved R11 10.2 mm to (157.6, 109.0), turned to 180 degrees
- moved R6 10.2 mm to (111.4, 107.3), turned to -90 degrees
- moved JP1 8.54 mm to (119.0, 97.4), turned to 180 degrees
- moved R14 3.20 mm to (147.4, 118.4)
- moved R15 3.20 mm to (147.4, 121.6)
- moved C13 3.01 mm to (153.8, 125.1)
- moved TP7 2.25 mm to (189.2, 121.8)
- moved JP3 1.09 mm to (134.7, 102.3)
- moved JP2 1.07 mm to (141.1, 102.3)
- moved C12 0.40 mm to (135.9, 124.3), turned to 0 degrees
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- renumbered C2 to C1, C13 to C10, C6 to C12, C9 to C13, C3 to C2, C5 to C3, C12 to C4, C10 to C5, C7 to C6, C4 to C7, C1 to C8, C8 to C9, D5 to D1, D7 to D10, D6 to D11, D4 to D2, D1 to D6, D10 to D7, D9 to D8, D8 to D9, J2 to J1, J3 to J2, J1 to J3, LK3 to LK1, LK1 to LK2, LK2 to LK3, Q1 to Q3, R10 to R1, R5 to R11, R14 to R13, R15 to R14, R16 to R15, R3 to R2, TP4 to TP1, TP1 to TP2, TP5 to TP3, TP6 to TP4, TP7 to TP5, TP2 to TP6, TP3 to TP7, U3 to U1, U1 to U3
Connections:
- D1 pad 1: Net-(D5-K) -> Net-(D1-K)
- D2 pad 1: Net-(D4-K) -> Net-(D2-K)
- D2 pad 2: Net-(D4-A) -> Net-(D2-A)
- JP2 pad 2: Net-(JP2-C) -> Net-(D2-K)
- JP2 pad 3: Net-(D4-K) -> Net-(JP2-B)
- JP3 pad 2: Net-(JP3-C) -> Net-(D3-K)
- JP3 pad 3: Net-(D3-K) -> Net-(JP3-B)
- LK1 pad 1: Net-(LK3-Pin_1) -> Net-(LK1-Pin_1)
- LK3 pad 1: Net-(LK2-Pin_1) -> Net-(LK3-Pin_1)
- R10 pad 2: Net-(R4-Pad2) -> Net-(D4-K)
- R11 pad 1: Net-(R4-Pad2) -> Net-(LK3-Pin_1)
- R11 pad 2: Net-(LK2-Pin_1) -> Net-(D4-K)
- R12 pad 1: Net-(R7-Pad2) -> +5V
- R12 pad 2: Net-(LK3-Pin_1) -> Net-(D5-K)
- R13 pad 1: Net-(R14-Pad1) -> Net-(D1-K)
- R5 pad 1: +5V -> Net-(D2-A)
- R5 pad 2: Net-(D4-A) -> +5V
- R6 pad 1: +5V -> Net-(D3-A)
- R6 pad 2: Net-(D3-A) -> +5V
- R8 pad 1: Net-(LK3-Pin_1) -> Net-(LK1-Pin_1)
- R8 pad 2: -15V -> Net-(D5-K)
- R9 pad 2: Net-(R7-Pad2) -> Net-(Q1-C)
- U1 pad 10: Net-(JP3-C) -> Net-(D3-K)
- U1 pad 11: Net-(JP2-C) -> Net-(D2-K)
- U1 pad 12: Net-(U3-R1OUT) -> Net-(U1-R1OUT)
- U2 pad 1: Net-(U3-R1OUT) -> Net-(U1-R1OUT)
- U2 pad 10: Net-(D3-K) -> Net-(JP3-B)
- U2 pad 11: Net-(R7-Pad2) -> Net-(Q1-C)
- U2 pad 12: Net-(D5-K) -> Net-(D1-K)
- U2 pad 13: Net-(U3-R1OUT) -> Net-(U2-Pad13)
- U2 pad 2: Net-(R14-Pad1) -> Net-(U2-Pad13)
- U2 pad 3: Net-(R4-Pad2) -> Net-(Q2-C)
- U2 pad 4: Net-(D4-K) -> Net-(JP2-B)
- U2 pad 5: Net-(D4-K) -> Net-(JP2-B)
- U2 pad 9: Net-(D3-K) -> Net-(JP3-B)
Routing:
- net Net-(D1-K): track 0.00 -> 73.1 mm
- net Net-(D2-K): track 0.00 -> 72.8 mm
- net Net-(LK2-Pin_1): track 68.4 -> 0.00 mm
- net GND: track 335.6 -> 393.8 mm
- net Net-(JP2-C): track 36.6 -> 0.00 mm
- net Net-(D4-K): track 68.6 -> 34.8 mm
- net Net-(U1-R1OUT): track 0.00 -> 31.9 mm
- net Net-(Q1-C): track 0.00 -> 31.5 mm
- net Net-(U3-R1OUT): track 30.6 -> 0.00 mm
- net Net-(R7-Pad2): track 28.8 -> 0.00 mm
- net Net-(JP3-C): track 26.4 -> 0.00 mm
- net -15V: track 264.4 -> 239.0 mm
- net Net-(Q2-C): track 0.00 -> 25.2 mm
- net Net-(R14-Pad1): track 24.8 -> 0.00 mm
- net Net-(LK1-Pin_1): track 0.00 -> 24.1 mm
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Other:
- board text added: "(c)Scott Finneran 2026 https://github.com/sierrafoxtrot"
- board text added: "2 3 8 5"
- board text added: "3 2 5 7"
- board text added: "3 7 Relay- 4 Relay+ 6"
- board text added: "3 TTI Return 7 TTO Relay- -15V 4 +10V Relay+ Reader Enable 6 TTO Return"
- board text added: "PDP-8 Serial AIO (DCE)"
- board text added: "PDP-8 Serial All-in-One"
- board text added: "RE"
- board text added: "Rx"
- board text added: "Serial Cable Wiring"
- board text added: "Terminal (25 way)"
- board text added: "Terminal (9 way)"
- board text added: "Tx"
- board text added: "W070 Current Loop"

Commit message: Revision A Hardware
Other:
- board text added: "CTS"
- board text added: "GND"
- board text added: "Rev. A"
- board text added: "Serial Cable"
- board text removed: "Serial Cable Wiring"
Changed lines of the file:
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@@
+		)
+	)
+	(gr_text "Rx"
+		(at 176 82.8 0)
+		(layer "B.SilkS")
+		(effects
+			(font
+				(size 0.746 0.746)
+				(thickness 0.1)
+			)
+			(justify left bottom mirror)
+		)
+	)
+	(gr_text "Tx"
+		(at 176 84.4 0)
+		(layer "B.SilkS")
+		(effects
+			(font
+				(size 0.746 0.746)
+				(thickness 0.1)
+			)
+			(justify left bottom mirror)
+		)
+	)
+	(gr_text "CTS"
+		(at 176 86 0)
+		(layer "B.SilkS")
+		(effects
+			(font
+				(size 0.746 0.746)
+				(thickness 0.1)
+			)
+			(justify left bottom mirror)
+		)
+	)
+	(gr_text "GND"
+		(at 176 87.6 0)
+		(layer "B.SilkS")
+		(effects
+			(font
+				(size 0.746 0.746)
+				(thickness 0.1)
+			)
+			(justify left bottom mirror)
+		)
+	)
+	(gr_text "Rev. A"
+		(at 95 130.587 0)
+		(layer "B.SilkS")
+		(effects
+			(font
+				(size 1 1)
+				(thickness 0.1)
+			)
+			(justify left bottom mirror)
 		)
 	)
@@
 		)
 	)
-	(gr_text "Serial Cable Wiring"
-		(at 163.8 81.4 0)
+	(gr_text "Serial Cable"
+		(at 165.4 81.4 0)
 		(layer "B.SilkS")
 		(effects
@@
 			)
 			(justify left bottom mirror)
+		)
+	)
+	(gr_text "PDP-8 Serial All-in-One"
+		(at 158.2 130.4 0)
+		(layer "B.SilkS")
+		(effects
+			(font
+				(size 1.5 1.5)
+				(thickness 0.3)
+				(bold yes)
+			)
+			(justify left bottom mirror)
