File: discrete/hardware/rx.kicad_sch (KiCad schematic)
At the start: 14 parts, among them Q4 2N5551, Q5 2N5401, Q6 2N5401

Commit message: Begin multi-sheet
Connections:
- net DEC_TTI renamed DEC_TTI_232
Changed lines of the file:
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@@
-	)
-	(junction
-		(at 72.39 100.33)
-		(diameter 0)
-		(color 0 0 0 0)
 	)
 	(junction
@@
 	(wire
 		(pts
-			(xy 59.69 97.79) (xy 59.69 100.33)
-		)
-		(stroke
-			(width 0)
-			(type default)
-		)
-	)
-	(wire
-		(pts
 			(xy 72.39 83.82) (xy 72.39 88.9)
 		)
@@
 	(wire
 		(pts
-			(xy 59.69 83.82) (xy 59.69 87.63)
-		)
-		(stroke
-			(width 0)
-			(type default)
-		)
-	)
-	(wire
-		(pts
 			(xy 182.88 104.14) (xy 182.88 105.41)
 		)
@@
 		(pts
 			(xy 83.82 83.82) (xy 87.63 83.82)
-		)
-		(stroke
-			(width 0)
-			(type default)
-		)
-	)
-	(wire
-		(pts
-			(xy 59.69 100.33) (xy 72.39 100.33)
 		)
 		(stroke
@@
 		)
 	)
-	(label "DEC_TTI"
-		(at 219.71 92.71 0)
+	(hierarchical_label "RS232_IN"
+		(shape input)
+		(at 59.69 83.82 180)
 		(effects
 			(font
 				(size 1.27 1.27)
 			)
-			(justify left bottom)
-		)
-	)
-	(label "RS232_IN"
-		(at 60.96 83.82 0)
+			(justify right)
+		)
+	)
+	(hierarchical_label "DEC_TTI_232"
+		(shape output)
+		(at 250.19 92.71 0)
 		(effects
 			(font
 				(size 1.27 1.27)
 			)
-			(justify left bottom)
-		)
-	)
+			(justify left)
+		)
+	)

Commit message: Laid out full schematic. Added decoupling and test points
Parts:
- added C6, C7: C, symbol Device:C
- added TP7, TP8: TestPoint, TestPoint:TestPoint_Loop_D3.50mm_Drill0.9mm_Beaded, symbol Connector:TestPoint
Connections:
- net +10V: now also C6.1
- net -15V: now also C7.2
- net GND: now also C6.2, C7.1
- net RX_SENSE: now also TP7.1
- net RX_SHIFT: now also TP8.1
Other:
- note added: "PDP-8 Serial All-in-One"
- note added: "RS-232 Receiver"
- moved on the sheet: R20
