File: discrete/hardware/PDP-8-Serial-Discrete.kicad_sch (KiCad schematic)
At the start: 27 parts, among them J1 Screw_Terminal_01x06, J2 DE9_Socket_MountingHoles, J3 FlipChip_01x18

Commit message: Geographic reannotation of PCB
Parts:
- renumbered C4 to C1, C3 to C2, C5 to C3, C2 to C4, C1 to C5, D4 to D5, R4 to R1, R1 to R13, R3 to R14, R2 to R15, R5 to R2, R6 to R3, TP6 to TP1, TP5 to TP2, TP4 to TP3, TP3 to TP4, TP1 to TP5, TP2 to TP6
Connections:
- net -15V: now also C4.1, R2.2; no longer C4.2, R2.1
- net GND: now also C4.2; no longer C4.1
- net TTI: now also R15.2; no longer R15.1
- net TTI_CL_RET: now also R2.1; no longer R2.2
- net at D2.1 (K): now also R15.1; no longer R15.2
Other:
- moved on the sheet: C4, R2
Changed lines of the file:
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@@
 		(on_board yes)
 		(dnp no)
-		(property "Reference" "TP2"
+		(property "Reference" "TP6"
 			(at 54.356 163.068 0)
 			(effects
@@
 			(project "PDP-8-Serial-Discrete"
 				(path "/b0fbf6eb-12c5-46d4-80aa-25b95de8bd79"
-					(reference "TP2")
+					(reference "TP6")
 					(unit 1)
 				)
@@
 	(symbol
 		(lib_id "Device:R")
-		(at 160.02 29.21 270)
-		(unit 1)
-		(exclude_from_sim no)
-		(in_bom yes)
-		(on_board yes)
-		(dnp no)
-		(property "Reference" "R5"
+		(at 160.02 29.21 90)
+		(mirror x)
+		(unit 1)
+		(exclude_from_sim no)
+		(in_bom yes)
+		(on_board yes)
+		(dnp no)
+		(property "Reference" "R2"
 			(at 160.02 29.21 90)
 			(effects
@@
 		)
 		(property "Value" "750R"
-			(at 157.988 31.75 90)
+			(at 158.242 31.75 90)
 			(effects
 				(font
@@
 			(project "PDP-8-Serial-Discrete"
 				(path "/b0fbf6eb-12c5-46d4-80aa-25b95de8bd79"
-					(reference "R5")
+					(reference "R2")
 					(unit 1)
 				)
@@
 		(on_board yes)
 		(dnp no)
-		(property "Reference" "C4"
+		(property "Reference" "C1"
 			(at 163.322 25.654 90)
 			(effects
@@
 			(project "PDP-8-Serial-Discrete"
 				(path "/b0fbf6eb-12c5-46d4-80aa-25b95de8bd79"
-					(reference "C4")
+					(reference "C1")
 					(unit 1)
 				)
@@
 		(on_board yes)
 		(dnp no)
-		(property "Reference" "D4"
+		(property "Reference" "D5"
 			(at 130.81 45.72 90)
 			(effects
@@
 			(project "PDP-8-Serial-Discrete"
 				(path "/b0fbf6eb-12c5-46d4-80aa-25b95de8bd79"
-					(reference "D4")
+					(reference "D5")
 					(unit 1)
 				)
@@
 		(dnp no)
 		(fields_autoplaced yes)
-		(property "Reference" "R1"
+		(property "Reference" "R13"
 			(at 29.21 33.0199 0)
 			(effects
@@
 			(project "PDP-8-Serial-Discrete"
 				(path "/b0fbf6eb-12c5-46d4-80aa-25b95de8bd79"
-					(reference "R1")
+					(reference "R13")
 					(unit 1)
 				)
@@
 		(on_board yes)
 		(dnp no)
-		(property "Reference" "TP5"
+		(property "Reference" "TP2"
 			(at 200.406 94.488 0)
 			(effects
@@
 			(project "PDP-8-Serial-Discrete"
 				(path "/b0fbf6eb-12c5-46d4-80aa-25b95de8bd79"
-					(reference "TP5")
+					(reference "TP2")
 					(unit 1)
 				)
@@
 		(on_board yes)
 		(dnp no)
-		(property "Reference" "TP3"
+		(property "Reference" "TP4"
 			(at 73.406 163.068 0)
 			(effects
@@
 			(project "PDP-8-Serial-Discrete"
 				(path "/b0fbf6eb-12c5-46d4-80aa-25b95de8bd79"
-					(reference "TP3")
+					(reference "TP4")
 					(unit 1)
 				)
@@
 		(lib_id "Device:R")
 		(at 41.91 34.29 0)
-		(unit 1)
-		(exclude_from_sim no)
-		(in_bom yes)
-		(on_board yes)
-		(dnp no)
-		(fields_autoplaced yes)
-		(property "Reference" "R2"
-			(at 44.45 33.0199 0)
+		(mirror x)
+		(unit 1)
+		(exclude_from_sim no)
+		(in_bom yes)
+		(on_board yes)
+		(dnp no)
+		(property "Reference" "R15"
+			(at 44.45 33.02 0)
 			(effects
 				(font
@@
 		)
 		(property "Value" "10k"
-			(at 44.45 35.5599 0)
+			(at 44.196 35.56 0)
 			(effects
 				(font
@@
 			(project "PDP-8-Serial-Discrete"
 				(path "/b0fbf6eb-12c5-46d4-80aa-25b95de8bd79"
-					(reference "R2")
+					(reference "R15")
 					(unit 1)
 				)
@@
 		(on_board yes)
 		(dnp no)
-		(property "Reference" "R4"
+		(property "Reference" "R1"
 			(at 144.78 33.02 90)
 			(effects
@@
 			(project "PDP-8-Serial-Discrete"
 				(path "/b0fbf6eb-12c5-46d4-80aa-25b95de8bd79"
-					(reference "R4")
+					(reference "R1")
 					(unit 1)
 				)
@@
 		(on_board yes)
 		(dnp no)
-		(property "Reference" "R6"
+		(property "Reference" "R3"
 			(at 182.88 45.72 90)
 			(effects
@@
 			(project "PDP-8-Serial-Discrete"
 				(path "/b0fbf6eb-12c5-46d4-80aa-25b95de8bd79"
-					(reference "R6")
+					(reference "R3")
 					(unit 1)
 				)
@@
 	(symbol
 		(lib_id "Device:C")
-		(at 63.5 168.91 90)
-		(unit 1)
-		(exclude_from_sim no)
-		(in_bom yes)
-		(on_board yes)
-		(dnp no)
-		(fields_autoplaced yes)
-		(property "Reference" "C2"
+		(at 63.5 168.91 270)
+		(mirror x)
+		(unit 1)
+		(exclude_from_sim no)
+		(in_bom yes)
+		(on_board yes)
+		(dnp no)
+		(property "Reference" "C4"
 			(at 63.5 161.29 90)
 			(effects
@@
 		)
 		(property "Footprint" "Capacitor_THT:C_Disc_D5.0mm_W2.5mm_P5.00mm"
-			(at 67.31 167.9448 0)
+			(at 59.69 167.9448 0)
 			(effects
 				(font
@@
 			(project "PDP-8-Serial-Discrete"
 				(path "/b0fbf6eb-12c5-46d4-80aa-25b95de8bd79"
-					(reference "C2")
+					(reference "C4")
 					(unit 1)
 				)
@@
 		(dnp no)
 		(fields_autoplaced yes)
-		(property "Reference" "C1"
+		(property "Reference" "C5"
 			(at 44.45 161.29 90)
 			(effects
@@
 			(project "PDP-8-Serial-Discrete"
 				(path "/b0fbf6eb-12c5-46d4-80aa-25b95de8bd79"
-					(reference "C1")
+					(reference "C5")
 					(unit 1)
 				)
@@
 		(on_board yes)
 		(dnp no)
-		(property "Reference" "C3"
+		(property "Reference" "C2"
 			(at 153.162 42.418 0)
 			(effects
@@
 			(project "PDP-8-Serial-Discrete"
 				(path "/b0fbf6eb-12c5-46d4-80aa-25b95de8bd79"
-					(reference "C3")
+					(reference "C2")
 					(unit 1)
 				)
@@
 		(on_board yes)
 		(dnp no)
-		(property "Reference" "TP1"
+		(property "Reference" "TP5"
 			(at 36.576 163.068 0)
 			(effects
@@
 			(project "PDP-8-Serial-Discrete"
 				(path "/b0fbf6eb-12c5-46d4-80aa-25b95de8bd79"
-					(reference "TP1")
+					(reference "TP5")
 					(unit 1)
 				)
@@
 		(dnp no)
 		(fields_autoplaced yes)
-		(property "Reference" "R3"
+		(property "Reference" "R14"
 			(at 59.69 33.0199 0)
 			(effects
@@
 			(project "PDP-8-Serial-Discrete"
 				(path "/b0fbf6eb-12c5-46d4-80aa-25b95de8bd79"
-					(reference "R3")
+					(reference "R14")
 					(unit 1)
 				)
@@
 		(on_board yes)
 		(dnp no)
-		(property "Reference" "TP4"
+		(property "Reference" "TP3"
 			(at 200.406 76.708 0)
 			(effects
@@
 			(project "PDP-8-Serial-Discrete"
 				(path "/b0fbf6eb-12c5-46d4-80aa-25b95de8bd79"
-					(reference "TP4")
+					(reference "TP3")
 					(unit 1)
 				)
@@
 		(on_board yes)
 		(dnp no)
-		(property "Reference" "TP6"
+		(property "Reference" "TP1"
 			(at 200.406 155.448 0)
 			(effects
@@
 			(project "PDP-8-Serial-Discrete"
 				(path "/b0fbf6eb-12c5-46d4-80aa-25b95de8bd79"
-					(reference "TP6")
+					(reference "TP1")
 					(unit 1)
 				)
@@
 		(on_board yes)
 		(dnp no)
-		(property "Reference" "C5"
+		(property "Reference" "C3"
 			(at 169.672 46.228 0)
 			(effects
@@
 			(project "PDP-8-Serial-Discrete"
 				(path "/b0fbf6eb-12c5-46d4-80aa-25b95de8bd79"
-					(reference "C5")
-					(unit 1)
-				)
+					(reference "C3")
+					(unit 1)
+				)

Commit message: Added BOM details
Parts:
- added H1, H2, H3, H4, H5: Jumper_Shunt, symbol Auxiliary_Items:Jumper_Shunt
- C1: DigiKey_PN (none) -> 2870-MKP1839510254-ND; MPN (none) -> MKP1839510254; Manufacturer (none) -> Vishay
- C2, C3: DigiKey_PN (none) -> 490-8812-ND; MPN (none) -> RDER71H103K0K1H03B; Manufacturer (none) -> Murata Electronics
- C4, C5: DigiKey_PN (none) -> 490-8816-ND; MPN (none) -> RDER71H105K2K1H03B; Manufacturer (none) -> Murata Electronics
- D1, D2, D3: DigiKey_PN (none) -> 160-1943-ND; MPN (none) -> LTL1CHKEKNN; Manufacturer (none) -> Lite-On
- D5: DigiKey_PN (none) -> 1N914B-ND; MPN (none) -> 1N914B; Manufacturer (none) -> onsemi
- J2: DigiKey_PN (none) -> AE10921-ND; MPN (none) -> A-DF 09 A/KG-T2S; Manufacturer (none) -> Assmann WSW Components
- J3, TP1, TP2, TP3, TP4, TP5, TP6: now left out of the parts list
- LK1, LK2, LK3: DigiKey_PN (none) -> S1012EC-03-ND; MPN (none) -> PREC003SAAAN-RC; Manufacturer (none) -> Sullins Connector Solutions
- R1: DigiKey_PN (none) -> 13-RSF100JB-73-1K-ND; MPN (none) -> RSF100JB-73-1K; Manufacturer (none) -> YAGEO
- R13, R14: DigiKey_PN (none) -> MFR-25FBF52-27K-ND; MPN (none) -> RES 27K OHM 1% 1/4W AXIAL; Manufacturer (none) -> YAGEO
- R15: DigiKey_PN (none) -> 10.0KXBK-ND; MPN (none) -> MFR-25FBF52-10K; Manufacturer (none) -> YAGEO
- R2, R3: DigiKey_PN (none) -> 13-RSF100JB-73-750R-ND; MPN (none) -> RSF100JB-73-750R; Manufacturer (none) -> YAGEO
