File: discrete/hardware/rs232_driver.kicad_sch (KiCad schematic)
At the start: 36 parts, among them J4 Conn_01x03, Q10 2N5401, Q11 2N5551, Q12 2N5401, Q7 2N5551, Q8 2N5401, Q9 2N5551

Commit message: Restructured for sheet reuse of rs232 driver. Annotated functional blocks of schematic. Resolved all ERC violations
Parts:
- removed DW1: 1N914, Diode_THT:D_DO-35_SOD27_P7.62mm_Horizontal, symbol Diode:1N914
- removed I1: 90m, symbol Simulation_SPICE:IDC
- removed QW1: 2N5401, Package_TO_SOT_THT:TO-92_Inline, symbol Transistor_BJT:2N3906
- removed RW1: 1k8, symbol Device:R
- removed RW2: 15k, symbol Device:R
- renumbered DW2 to D4, D14 to D5, D15 to D6, D16 to D7, D17 to D8, D18 to D9, Q12 to Q10, QW2 to Q4, Q7 to Q5, Q8 to Q6, Q9 to Q7, Q10 to Q8, Q11 to Q9, RW3 to R13, RW4 to R14, RW5 to R15, RW6 to R16, R25 to R17, R26 to R18, R27 to R19, R28 to R20, R29 to R21, R30 to R22, R31 to R23, R32 to R24, R33 to R25, R34 to R26, TP10 to TP12
Connections:
- net DEC_TTO_232 renamed DEC_IN
- net TTO_INV renamed DEC_IN_INV
Other:
- note added: "${SHEETNAME} (RS232 Driver)"
- note added: "INVERTER"
- note added: "LEVEL CONVERTER"
- note added: "NEGATIVE LINE DRIVER"
- note added: "POSITIVE LINE DRIVER"
- note added: "SWITCHING AMPLIFIER"
- note removed: "RS-232 Transmitter"
- moved on the sheet: J4

Commit message: Set footprints and component ratings
Parts:
- C8, C9: footprint (none) -> Capacitor_THT:C_Disc_D5.0mm_W2.5mm_P2.50mm
- J4: footprint (none) -> Connector_PinHeader_2.54mm:PinHeader_1x03_P2.54mm_Vertical
- R13, R14, R15, R16, R17, R18, R19, R20, R21, R22, R23, R24, R25, R26: footprint (none) -> Resistor_THT:R_Axial_DIN0207_L6.3mm_D2.5mm_P10.16mm_Horizontal
Changed lines of the file:
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@@
 			)
 		)
-		(property "Footprint" ""
+		(property "Footprint" "Resistor_THT:R_Axial_DIN0207_L6.3mm_D2.5mm_P10.16mm_Horizontal"
 			(at 102.87 89.408 90)
 			(effects
@@
 			)
 		)
-		(property "Footprint" ""
+		(property "Footprint" "Resistor_THT:R_Axial_DIN0207_L6.3mm_D2.5mm_P10.16mm_Horizontal"
 			(at 190.5 93.218 90)
 			(effects
@@
 			)
 		)
-		(property "Footprint" ""
+		(property "Footprint" "Resistor_THT:R_Axial_DIN0207_L6.3mm_D2.5mm_P10.16mm_Horizontal"
 			(at 134.112 74.93 90)
 			(effects
@@
 			)
 		)
-		(property "Footprint" ""
+		(property "Footprint" "Capacitor_THT:C_Disc_D5.0mm_W2.5mm_P2.50mm"
 			(at 47.2948 173.99 0)
 			(effects
@@
 			)
 		)
-		(property "Footprint" ""
+		(property "Footprint" "Connector_PinHeader_2.54mm:PinHeader_1x03_P2.54mm_Vertical"
 			(at 88.9 76.2 0)
 			(effects
@@
 			)
 		)
-		(property "Footprint" ""
+		(property "Footprint" "Resistor_THT:R_Axial_DIN0207_L6.3mm_D2.5mm_P10.16mm_Horizontal"
 			(at 57.912 68.58 90)
 			(effects
@@
 			)
 		)
-		(property "Footprint" ""
+		(property "Footprint" "Resistor_THT:R_Axial_DIN0207_L6.3mm_D2.5mm_P10.16mm_Horizontal"
 			(at 70.612 68.58 90)
 			(effects
@@
 			)
 		)
-		(property "Footprint" ""
+		(property "Footprint" "Resistor_THT:R_Axial_DIN0207_L6.3mm_D2.5mm_P10.16mm_Horizontal"
 			(at 214.122 80.01 90)
 			(effects
@@
 			)
 		)
-		(property "Footprint" ""
+		(property "Footprint" "Resistor_THT:R_Axial_DIN0207_L6.3mm_D2.5mm_P10.16mm_Horizontal"
 			(at 168.402 97.79 90)
 			(effects
@@
 			)
 		)
-		(property "Footprint" ""
+		(property "Footprint" "Resistor_THT:R_Axial_DIN0207_L6.3mm_D2.5mm_P10.16mm_Horizontal"
 			(at 52.07 93.218 90)
 			(effects
@@
 			)
 		)
-		(property "Footprint" ""
+		(property "Footprint" "Resistor_THT:R_Axial_DIN0207_L6.3mm_D2.5mm_P10.16mm_Horizontal"
 			(at 108.712 77.47 90)
 			(effects
@@
 			)
 		)
-		(property "Footprint" ""
+		(property "Footprint" "Resistor_THT:R_Axial_DIN0207_L6.3mm_D2.5mm_P10.16mm_Horizontal"
 			(at 44.958 120.65 90)
 			(effects
@@
 			)
 		)
-		(property "Footprint" ""
+		(property "Footprint" "Resistor_THT:R_Axial_DIN0207_L6.3mm_D2.5mm_P10.16mm_Horizontal"
 			(at 190.5 75.438 90)
 			(effects
@@
 			)
 		)
-		(property "Footprint" ""
+		(property "Footprint" "Resistor_THT:R_Axial_DIN0207_L6.3mm_D2.5mm_P10.16mm_Horizontal"
 			(at 214.122 90.17 90)
 			(effects
@@
 			)
 		)
-		(property "Footprint" ""
+		(property "Footprint" "Capacitor_THT:C_Disc_D5.0mm_W2.5mm_P2.50mm"
 			(at 64.77 175.5648 0)
 			(effects
@@
 			)
 		)
-		(property "Footprint" ""
+		(property "Footprint" "Resistor_THT:R_Axial_DIN0207_L6.3mm_D2.5mm_P10.16mm_Horizontal"
 			(at 153.162 72.39 90)
 			(effects
@@
 			)
 		)
-		(property "Footprint" ""
+		(property "Footprint" "Resistor_THT:R_Axial_DIN0207_L6.3mm_D2.5mm_P10.16mm_Horizontal"
 			(at 147.32 83.058 90)
 			(effects

Commit message: Added holeless flip-chip layout. Footprints assigned.
Parts:
- R13, R14, R15, R16, R17, R18, R19, R20, R21, R22, R23, R24, R25, R26: footprint Resistor_THT:R_Axial_DIN0207_L6.3mm_D2.5mm_P10.16mm_Horizontal -> Resistor_THT:R_Axial_DIN0207_L6.3mm_D2.5mm_P7.62mm_Horizontal
Changed lines of the file:
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@@
 			)
 		)
-		(property "Footprint" "Resistor_THT:R_Axial_DIN0207_L6.3mm_D2.5mm_P10.16mm_Horizontal"
+		(property "Footprint" "Resistor_THT:R_Axial_DIN0207_L6.3mm_D2.5mm_P7.62mm_Horizontal"
 			(at 102.87 89.408 90)
 			(effects
@@
 			)
 		)
-		(property "Footprint" "Resistor_THT:R_Axial_DIN0207_L6.3mm_D2.5mm_P10.16mm_Horizontal"
+		(property "Footprint" "Resistor_THT:R_Axial_DIN0207_L6.3mm_D2.5mm_P7.62mm_Horizontal"
 			(at 190.5 93.218 90)
 			(effects
@@
 			)
 		)
-		(property "Footprint" "Resistor_THT:R_Axial_DIN0207_L6.3mm_D2.5mm_P10.16mm_Horizontal"
+		(property "Footprint" "Resistor_THT:R_Axial_DIN0207_L6.3mm_D2.5mm_P7.62mm_Horizontal"
 			(at 134.112 74.93 90)
 			(effects
@@
 			)
 		)
-		(property "Footprint" "Resistor_THT:R_Axial_DIN0207_L6.3mm_D2.5mm_P10.16mm_Horizontal"
+		(property "Footprint" "Resistor_THT:R_Axial_DIN0207_L6.3mm_D2.5mm_P7.62mm_Horizontal"
 			(at 57.912 68.58 90)
 			(effects
@@
 			)
 		)
-		(property "Footprint" "Resistor_THT:R_Axial_DIN0207_L6.3mm_D2.5mm_P10.16mm_Horizontal"
+		(property "Footprint" "Resistor_THT:R_Axial_DIN0207_L6.3mm_D2.5mm_P7.62mm_Horizontal"
 			(at 70.612 68.58 90)
 			(effects
@@
 			)
 		)
-		(property "Footprint" "Resistor_THT:R_Axial_DIN0207_L6.3mm_D2.5mm_P10.16mm_Horizontal"
+		(property "Footprint" "Resistor_THT:R_Axial_DIN0207_L6.3mm_D2.5mm_P7.62mm_Horizontal"
 			(at 214.122 80.01 90)
 			(effects
@@
 			)
 		)
-		(property "Footprint" "Resistor_THT:R_Axial_DIN0207_L6.3mm_D2.5mm_P10.16mm_Horizontal"
+		(property "Footprint" "Resistor_THT:R_Axial_DIN0207_L6.3mm_D2.5mm_P7.62mm_Horizontal"
 			(at 168.402 97.79 90)
 			(effects
@@
 			)
 		)
-		(property "Footprint" "Resistor_THT:R_Axial_DIN0207_L6.3mm_D2.5mm_P10.16mm_Horizontal"
+		(property "Footprint" "Resistor_THT:R_Axial_DIN0207_L6.3mm_D2.5mm_P7.62mm_Horizontal"
 			(at 52.07 93.218 90)
 			(effects
@@
 			)
 		)
-		(property "Footprint" "Resistor_THT:R_Axial_DIN0207_L6.3mm_D2.5mm_P10.16mm_Horizontal"
+		(property "Footprint" "Resistor_THT:R_Axial_DIN0207_L6.3mm_D2.5mm_P7.62mm_Horizontal"
 			(at 108.712 77.47 90)
 			(effects
@@
 			)
 		)
-		(property "Footprint" "Resistor_THT:R_Axial_DIN0207_L6.3mm_D2.5mm_P10.16mm_Horizontal"
+		(property "Footprint" "Resistor_THT:R_Axial_DIN0207_L6.3mm_D2.5mm_P7.62mm_Horizontal"
 			(at 44.958 120.65 90)
 			(effects
@@
 			)
 		)
-		(property "Footprint" "Resistor_THT:R_Axial_DIN0207_L6.3mm_D2.5mm_P10.16mm_Horizontal"
+		(property "Footprint" "Resistor_THT:R_Axial_DIN0207_L6.3mm_D2.5mm_P7.62mm_Horizontal"
 			(at 190.5 75.438 90)
 			(effects
@@
 			)
 		)
-		(property "Footprint" "Resistor_THT:R_Axial_DIN0207_L6.3mm_D2.5mm_P10.16mm_Horizontal"
+		(property "Footprint" "Resistor_THT:R_Axial_DIN0207_L6.3mm_D2.5mm_P7.62mm_Horizontal"
 			(at 214.122 90.17 90)
 			(effects
@@
 			)
 		)
-		(property "Footprint" "Resistor_THT:R_Axial_DIN0207_L6.3mm_D2.5mm_P10.16mm_Horizontal"
+		(property "Footprint" "Resistor_THT:R_Axial_DIN0207_L6.3mm_D2.5mm_P7.62mm_Horizontal"
 			(at 153.162 72.39 90)
 			(effects
@@
 			)
 		)
-		(property "Footprint" "Resistor_THT:R_Axial_DIN0207_L6.3mm_D2.5mm_P10.16mm_Horizontal"
+		(property "Footprint" "Resistor_THT:R_Axial_DIN0207_L6.3mm_D2.5mm_P7.62mm_Horizontal"
 			(at 147.32 83.058 90)
 			(effects

Commit message: New footprints and symbols. PCB layout begun
Parts:
- removed J4: Conn_01x03, Connector_PinHeader_2.54mm:PinHeader_1x03_P2.54mm_Vertical, symbol Connector_Generic:Conn_01x03
- removed TP12: TestPoint, TestPoint:TestPoint_Loop_D3.50mm_Drill0.9mm_Beaded, symbol Connector:TestPoint
- added LK4: Link_01x03, Connector_PinHeader_2.54mm:PinHeader_1x03_P2.54mm_Vertical, symbol Links:Link_01x03
- renumbered D7 to D10, D8 to D11, D9 to D12, D4 to D7, D5 to D8, D6 to D9, R13 to R16, R14 to R17, R15 to R18, R16 to R19, R17 to R20, R18 to R21, R19 to R22, R20 to R23, R21 to R24, R22 to R25, R23 to R26, R24 to R27, R25 to R28, R26 to R29
Connections:
- net DEC_IN: now also LK4.3 (Pin_3)
- net DEC_IN_INV: now also LK4.1 (Pin_1)
- net at R20.1: now also LK4.2 (Pin_2)

Commit message: Geographic reannotation of PCB
Parts:
- renumbered C9 to C8, C8 to C9, D12 to D10, D8 to D11, D7 to D12, D10 to D7, D9 to D8, D11 to D9, Q4 to Q10, Q10 to Q4, Q8 to Q5, Q9 to Q6, Q5 to Q8, Q6 to Q9, R28 to R16, R29 to R17, R26 to R18, R25 to R19, R27 to R20, R24 to R21, R23 to R22, R22 to R23, R21 to R24, R20 to R25, R17 to R26, R16 to R27, R18 to R28, R19 to R29
Connections:
- net +10V: now also R28.1; no longer R28.2
- net -15V: now also R29.1; no longer R29.2
- net DEC_IN: now also R26.2; no longer R26.1
- net DEC_IN_INV: now also R29.2; no longer R29.1
- net Q3_E: now also R16.2; no longer R16.1
- net RS232_OUT: now also R16.1; no longer R16.2
- net at D12.2 (A), Q10.2 (B): now also R26.1, R28.2; no longer R26.2, R28.1
Other:
- moved on the sheet: R26

Commit message: Added BOM details
Parts:
- C8, C9: DigiKey_PN (none) -> 490-9145-1-ND; MPN (none) -> RDER71H104K0S1H03A; Manufacturer (none) -> Murata Electronics
- D10, D11, D12, D7, D8, D9: DigiKey_PN (none) -> 1N914B-ND; MPN (none) -> 1N914B; Manufacturer (none) -> onsemi
- LK4: DigiKey_PN (none) -> S1012EC-03-ND; MPN (none) -> PREC003SAAAN-RC; Manufacturer (none) -> Sullins Connector Solutions
- Q10, Q4, Q5, Q9: DigiKey_PN (none) -> 4878-2N5401CT-ND; MPN (none) -> 2N5401; Manufacturer (none) -> Diotec Semiconductor
- Q6, Q7, Q8: DigiKey_PN (none) -> 4878-2N5551CT-ND; MPN (none) -> 2N5551; Manufacturer (none) -> Diotec Semiconductor
- R16, R17: DigiKey_PN (none) -> 13-MFR-25FBF52-68R-ND; MPN (none) -> RES 68 OHM 1% 1/4W AXIAL; Manufacturer (none) -> YAGEO
- R18, R19, R20, R29: DigiKey_PN (none) -> 10.0KXBK-ND; MPN (none) -> MFR-25FBF52-10K; Manufacturer (none) -> YAGEO
- R21, R23, R28: DigiKey_PN (none) -> 100KXBK-ND; MPN (none) -> MFR-25FBF52-100K; Manufacturer (none) -> YAGEO
- R22: DigiKey_PN (none) -> RES 68 OHM 1% 1/4W AXIAL; MPN (none) -> MFR-25FBF52-33K; Manufacturer (none) -> YAGEO
- R24, R26: DigiKey_PN (none) -> MFR-25FBF52-47K-ND; MPN (none) -> RES 47K OHM 1% 1/4W AXIAL; Manufacturer (none) -> YAGEO
- R25: DigiKey_PN (none) -> MFR-25FBF52-27K-ND; MPN (none) -> RES 27K OHM 1% 1/4W AXIAL; Manufacturer (none) -> YAGEO
- R27: DigiKey_PN (none) -> 7.50KXBK-ND; MPN (none) -> RES 7.5K OHM 1% 1/4W AXIAL; Manufacturer (none) -> YAGEO
