File: discrete/hardware/PDP-8-Serial-Discrete.kicad_pcb (KiCad board)
At the start: 2 copper layers, 125.7 x 62.2 mm, 61 parts, among them J1 Screw_Terminal_01x06, J2 DE9_Socket_MountingHoles, J3 FlipChip_01x18, Q1 2N3904, Q2 2N3904, Q3 2N3906, U1 MAX232, U2 74HCT14, U3 L78L05_TO92

Commit message: Started PCB
Parts:
- removed C12, C13: 100nF, Capacitor_THT:C_Disc_D5.0mm_W2.5mm_P2.50mm
- removed JP1: SolderJumper_2_Bridged, Jumper:SolderJumper-2_P1.3mm_Bridged2Bar_RoundedPad1.0x1.5mm
- removed JP2, JP3: SolderJumper_3_Bridged12, Jumper:SolderJumper-3_P1.3mm_Bridged2Bar12_RoundedPad1.0x1.5mm_NumberLabels
- removed U1: MAX232, Package_DIP:DIP-16_W7.62mm
- removed U2: 74HCT14, Package_DIP:DIP-14_W7.62mm
- removed U3: L78L05_TO92, Package_TO_SOT_THT:TO-92_Inline
- added D12: 1N914, Diode_THT:D_DO-35_SOD27_P7.62mm_Horizontal, F.Cu at (96.7, 30.9)
- added D13: 1N914, Diode_THT:D_DO-35_SOD27_P7.62mm_Horizontal, F.Cu at (100.3, 30.9)
- added D14: 1N914, Diode_THT:D_DO-35_SOD27_P7.62mm_Horizontal, F.Cu at (103.8, 30.9)
- added D15: 1N914, Diode_THT:D_DO-35_SOD27_P7.62mm_Horizontal, F.Cu at (107.4, 30.9)
- added J4: Conn_01x03, Connector_PinHeader_2.54mm:PinHeader_1x03_P2.54mm_Vertical, F.Cu at (148.9, 19.5)
- added J5: Conn_01x03, Connector_PinHeader_2.54mm:PinHeader_1x03_P2.54mm_Vertical, F.Cu at (90.2, 19.5)
- added Q10: 2N5401, Package_TO_SOT_THT:TO-92_Inline, F.Cu at (138.2, 24.0)
- added Q11: 2N5401, Package_TO_SOT_THT:TO-92_Inline, F.Cu at (68.0, 30.5)
- added Q12: 2N5551, Package_TO_SOT_THT:TO-92_Inline, F.Cu at (73.8, 30.5)
- added Q13: 2N5401, Package_TO_SOT_THT:TO-92_Inline, F.Cu at (79.5, 30.5)
- added Q14: 2N5551, Package_TO_SOT_THT:TO-92_Inline, F.Cu at (85.3, 30.5)
- added Q15: 2N5401, Package_TO_SOT_THT:TO-92_Inline, F.Cu at (68.0, 24.0)
- added Q16: 2N5551, Package_TO_SOT_THT:TO-92_Inline, F.Cu at (73.8, 24.0)
- added Q17: 2N5401, Package_TO_SOT_THT:TO-92_Inline, F.Cu at (79.5, 24.0)
- added Q4: 2N5401, Package_TO_SOT_THT:TO-92_Inline, F.Cu at (126.7, 30.5)
- added Q5: 2N5551, Package_TO_SOT_THT:TO-92_Inline, F.Cu at (132.5, 30.5)
- added Q6: 2N5401, Package_TO_SOT_THT:TO-92_Inline, F.Cu at (138.2, 30.5)
- added Q7: 2N5551, Package_TO_SOT_THT:TO-92_Inline, F.Cu at (144.0, 30.5)
- added Q8: 2N5401, Package_TO_SOT_THT:TO-92_Inline, F.Cu at (126.7, 24.0)
- added Q9: 2N5551, Package_TO_SOT_THT:TO-92_Inline, F.Cu at (132.5, 24.0)
- added R16: 10k, Resistor_THT:R_Axial_DIN0207_L6.3mm_D2.5mm_P10.16mm_Horizontal, F.Cu at (137.6, 44.3)
- added R17: 27k, Resistor_THT:R_Axial_DIN0207_L6.3mm_D2.5mm_P10.16mm_Horizontal, F.Cu at (141.6, 44.3)
- added R18: 47k, Resistor_THT:R_Axial_DIN0207_L6.3mm_D2.5mm_P10.16mm_Horizontal, F.Cu at (145.7, 44.3)
- added R19: 100k, Resistor_THT:R_Axial_DIN0207_L6.3mm_D2.5mm_P10.16mm_Horizontal, F.Cu at (149.7, 44.3)
- added R20: 33k, Resistor_THT:R_Axial_DIN0207_L6.3mm_D2.5mm_P10.16mm_Horizontal, F.Cu at (153.8, 44.3)
- added R21: 100k, Resistor_THT:R_Axial_DIN0207_L6.3mm_D2.5mm_P10.16mm_Horizontal, F.Cu at (157.8, 44.3)
- added R22: 10k, Resistor_THT:R_Axial_DIN0207_L6.3mm_D2.5mm_P10.16mm_Horizontal, F.Cu at (161.9, 44.3)
- added R23: 10k, Resistor_THT:R_Axial_DIN0207_L6.3mm_D2.5mm_P10.16mm_Horizontal, F.Cu at (165.9, 44.3)
- added R24: 10k, Resistor_THT:R_Axial_DIN0207_L6.3mm_D2.5mm_P10.16mm_Horizontal, F.Cu at (170.0, 44.3)
- added R25: 68, Resistor_THT:R_Axial_DIN0207_L6.3mm_D2.5mm_P10.16mm_Horizontal, F.Cu at (174.0, 44.3)
- added R26: 68, Resistor_THT:R_Axial_DIN0207_L6.3mm_D2.5mm_P10.16mm_Horizontal, F.Cu at (178.1, 44.3)
- added R27: 7k5, Resistor_THT:R_Axial_DIN0207_L6.3mm_D2.5mm_P10.16mm_Horizontal, F.Cu at (66.7, 44.3)
- added R28: 47k, Resistor_THT:R_Axial_DIN0207_L6.3mm_D2.5mm_P10.16mm_Horizontal, F.Cu at (70.8, 44.3)
- added R29: 100k, Resistor_THT:R_Axial_DIN0207_L6.3mm_D2.5mm_P10.16mm_Horizontal, F.Cu at (74.8, 44.3)
- added R30: 10k, Resistor_THT:R_Axial_DIN0207_L6.3mm_D2.5mm_P10.16mm_Horizontal, F.Cu at (78.9, 44.3)
- added R31: 27k, Resistor_THT:R_Axial_DIN0207_L6.3mm_D2.5mm_P10.16mm_Horizontal, F.Cu at (82.9, 44.3)
- added R32: 47k, Resistor_THT:R_Axial_DIN0207_L6.3mm_D2.5mm_P10.16mm_Horizontal, F.Cu at (87.0, 44.3)
- added R33: 100k, Resistor_THT:R_Axial_DIN0207_L6.3mm_D2.5mm_P10.16mm_Horizontal, F.Cu at (91.0, 44.3)
- added R34: 33k, Resistor_THT:R_Axial_DIN0207_L6.3mm_D2.5mm_P10.16mm_Horizontal, F.Cu at (95.1, 44.3)
- added R35: 100k, Resistor_THT:R_Axial_DIN0207_L6.3mm_D2.5mm_P10.16mm_Horizontal, F.Cu at (99.1, 44.3)
- added R36: 10k, Resistor_THT:R_Axial_DIN0207_L6.3mm_D2.5mm_P10.16mm_Horizontal, F.Cu at (103.2, 44.3)
- added R37: 10k, Resistor_THT:R_Axial_DIN0207_L6.3mm_D2.5mm_P10.16mm_Horizontal, F.Cu at (107.2, 44.3)
- added R38: 10k, Resistor_THT:R_Axial_DIN0207_L6.3mm_D2.5mm_P10.16mm_Horizontal, F.Cu at (111.3, 44.3)
- added R39: 68, Resistor_THT:R_Axial_DIN0207_L6.3mm_D2.5mm_P10.16mm_Horizontal, F.Cu at (115.3, 44.3)
- added R40: 68, Resistor_THT:R_Axial_DIN0207_L6.3mm_D2.5mm_P10.16mm_Horizontal, F.Cu at (119.4, 44.3)
- added TP10: TestPoint, TestPoint:TestPoint_Loop_D3.50mm_Drill0.9mm_Beaded, F.Cu at (184.7, 23.4)
- added TP11: TestPoint, TestPoint:TestPoint_Loop_D3.50mm_Drill0.9mm_Beaded, F.Cu at (190.0, 23.4)
- added TP12: TestPoint, TestPoint:TestPoint_Loop_D3.50mm_Drill0.9mm_Beaded, F.Cu at (170.5, 23.3)
- added TP13: TestPoint, TestPoint:TestPoint_Loop_D3.50mm_Drill0.9mm_Beaded, F.Cu at (111.8, 23.3)
- added TP8: TTI, TestPoint:TestPoint_Loop_D3.50mm_Drill0.9mm_Beaded, F.Cu at (138.7, 73.7)
- added TP9: TTI, TestPoint:TestPoint_Loop_D3.50mm_Drill0.9mm_Beaded, F.Cu at (144.0, 73.7)
- C1: value 10nF -> 1uF; footprint Capacitor_THT:C_Disc_D5.0mm_W2.5mm_P2.50mm -> Capacitor_THT:C_Disc_D5.0mm_W2.5mm_P5.00mm
- C11, C6, C9: value 1uF -> 100nF; footprint Capacitor_THT:C_Disc_D5.0mm_W2.5mm_P5.00mm -> Capacitor_THT:C_Disc_D5.0mm_W2.5mm_P2.50mm
- C2: value 1uF 150VDC -> 1uF; footprint Capacitor_THT:CP_Axial_L29.0mm_D13.0mm_P35.00mm_Horizontal -> Capacitor_THT:C_Disc_D5.0mm_W2.5mm_P5.00mm
- C4: value 1uF -> 1uF 150VDC; footprint Capacitor_THT:C_Disc_D5.0mm_W2.5mm_P5.00mm -> Capacitor_THT:CP_Axial_L29.0mm_D13.0mm_P35.00mm_Horizontal
- C5: value 1uF -> 10nF; footprint Capacitor_THT:C_Disc_D5.0mm_W2.5mm_P5.00mm -> Capacitor_THT:C_Disc_D5.0mm_W2.5mm_P2.50mm
- C8: value 330nF -> 100nF; footprint Capacitor_THT:C_Disc_D5.0mm_W2.5mm_P5.00mm -> Capacitor_THT:C_Disc_D5.0mm_W2.5mm_P2.50mm
- D1, D2, D3: value LED -> 1N914; footprint LED_THT:LED_D3.0mm -> Diode_THT:D_DO-35_SOD27_P7.62mm_Horizontal
- J3: footprint DEC:FlipChip_SingleSided_CardEdge -> Connector_PCBEdge:DEC_single_short
- Q1: value 2N3904 -> 2N5551
- Q2: value 2N3904 -> 2N5401
- Q3: value 2N3906 -> 2N5401
- R1: value 750R 1W -> 1k
- R10: value 330k -> 10k
- R11: value 100k -> 2k7
- R12: value 330k -> 2k2
- R13: value 10k -> 7k5
- R14: value 1k -> 47k
- R15: value 3k -> 100k
- R2: value 750R 1W -> 750R
- R3: value 1k -> 750R; footprint Resistor_THT:R_Axial_DIN0207_L6.3mm_D2.5mm_P10.16mm_Horizontal -> Resistor_THT:R_Axial_DIN0414_L11.9mm_D4.5mm_P20.32mm_Horizontal
- R4: value 1k -> 5k1
- R5: value 1k -> 100k
- R6: value 1k -> 470k
- R8: value 100k -> 47k
- TP1: value -15V -> TTI
- TP2: value GND -> TTI
- TP6: value +5V -> TTI
- TP7: value +10V -> TTI
- moved D2 129.2 mm to (209.4, 30.9), turned to 90 degrees
- moved D3 127.7 mm to (212.9, 30.9), turned to 90 degrees
- moved D10 123.9 mm to (89.6, 30.9), turned to 90 degrees
- moved D11 123.1 mm to (93.2, 30.9), turned to 90 degrees
- moved C6 112.0 mm to (201.5, 30.5), turned to 90 degrees
- moved R4 107.8 mm to (184.1, 44.3)
- moved C9 106.2 mm to (173.9, 30.5), turned to 90 degrees
- moved R6 102.5 mm to (192.2, 44.3), turned to 90 degrees
- moved R5 101.9 mm to (188.2, 44.3), turned to 90 degrees
- moved Q3 95.8 mm to (196.9, 30.5), turned to 90 degrees
- moved C10 95.7 mm to (111.2, 30.5), turned to 90 degrees
- moved C7 94.9 mm to (205.6, 30.5), turned to 90 degrees
- moved C11 92.2 mm to (115.2, 30.5), turned to 90 degrees
- moved C8 90.4 mm to (169.9, 30.5), turned to 90 degrees
- moved R12 89.9 mm to (216.5, 44.3), turned to 90 degrees
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Connections:
- net /<NO NET> renamed /DSR
- C1 pad 1: /TTO_CL -> +10V
- C10 pad 1: +5V -> +10V
- C11 pad 1: Net-(U1-VS+) -> GND
- C11 pad 2: GND -> -15V
- C2 pad 1: /TTI_CL_RET -> GND
- C3 pad 1: /RDR_EN_CL -> /TTO_CL
- C4 pad 1: Net-(U1-VS-) -> /TTI_CL_RET
- C4 pad 2: GND -> -15V
- C5 pad 1: Net-(U1-C2-) -> /RDR_EN_CL
- C5 pad 2: Net-(U1-C2+) -> GND
- C6 pad 1: Net-(U1-C1-) -> +10V
- C6 pad 2: Net-(U1-C1+) -> GND
- C7 pad 1: +5V -> GND
- C7 pad 2: GND -> -15V
- C9 pad 1: +5V -> GND
- C9 pad 2: GND -> -15V
- D1 pad 1: Net-(D1-K) -> GND
- D1 pad 2: Net-(D1-A) -> /TTI_CL
- D10 pad 1: Net-(D10-K) -> GND
- D11 pad 1: Net-(D10-A) -> Net-(D11-K)
- D2 pad 2: Net-(D2-A) -> GND
- D3 pad 1: Net-(D3-K) -> GND
- D4 pad 1: Net-(D4-K) -> GND
- D4 pad 2: GND -> Net-(D4-A)
- D6 pad 1: GND -> Net-(D6-K)
- D6 pad 2: /TTI_CL -> /Transmitter/B3
- D7 pad 1: /TTI_EIA_NEG -> /Transmitter/B4
- D8 pad 1: Net-(D7-A) -> /Transmitter/B3
- D8 pad 2: Net-(D8-A) -> /Transmitter/Q3_E
- D9 pad 1: Net-(D8-A) -> /Transmitter/Q4_E
- D9 pad 2: Net-(D10-K) -> /Transmitter/B4
- LK1 pad 1: Net-(LK1-Pin_1) -> /TTI_EIA_NEG
- LK1 pad 2: /RDR_EN -> /TTI
- LK1 pad 3: /RDR_EN_CL -> /TTI_CL
- LK2 pad 1: /TTI_EIA_NEG -> /DEC_TTO_232
- LK2 pad 2: /TTI -> /TTO
- LK2 pad 3: /TTI_CL -> /TTO_CL
- LK3 pad 1: Net-(LK3-Pin_1) -> /DEC_REN_232
- LK3 pad 2: /TTO -> /RDR_EN
- LK3 pad 3: /TTO_CL -> /RDR_EN_CL
- Q1 pad 2: Net-(D5-K) -> Net-(D2-K)
- Q1 pad 3: Net-(Q1-C) -> /Receiver/RX_SENSE
- Q2 pad 1: GND -> +10V
- Q2 pad 2: Net-(D4-K) -> Net-(Q2-B)
- Q2 pad 3: Net-(Q2-C) -> /Receiver/RX_SHIFT
- Q3 pad 1: +5V -> GND
- Q3 pad 2: Net-(Q3-B) -> Net-(D3-A)
- Q3 pad 3: Net-(Q3-C) -> /TTI_EIA_NEG
- R1 pad 1: /TTO_CL_RET -> /TTI_CL_RET
- R1 pad 2: -15V -> /TTI_CL
- R10 pad 1: +5V -> /Receiver/RX_SHIFT
- R10 pad 2: Net-(D4-K) -> Net-(D3-A)
- R11 pad 1: Net-(LK3-Pin_1) -> /TTI_EIA_NEG
- R11 pad 2: Net-(D4-K) -> GND
- R12 pad 1: +5V -> /TTI_EIA_NEG
- R12 pad 2: Net-(D5-K) -> -15V
- R13 pad 1: Net-(D1-K) -> -15V
- R13 pad 2: Net-(Q3-B) -> /DEC_TTO_232
- R14 pad 1: /TTI_EIA_NEG -> /DEC_TTO_232
- R14 pad 2: Net-(Q3-C) -> Net-(D4-A)
- R15 pad 1: /TTI_EIA_NEG -> Net-(D4-A)
- R15 pad 2: -15V -> +10V
- R3 pad 1: /TTI_CL_RET -> /TTO_CL_RET
- R3 pad 2: /TTI_CL -> -15V
- R4 pad 1: +5V -> GND
- R4 pad 2: Net-(D1-A) -> /TxD
- R5 pad 1: Net-(D2-A) -> /TxD
- R5 pad 2: +5V -> Net-(D2-K)
- R6 pad 1: Net-(D3-A) -> GND
- R6 pad 2: +5V -> Net-(D2-K)
- R7 pad 1: +5V -> /Receiver/RX_SENSE
- R7 pad 2: Net-(Q2-C) -> +10V
- R8 pad 1: Net-(LK1-Pin_1) -> Net-(Q2-B)
- R8 pad 2: Net-(D5-K) -> /Receiver/RX_SENSE
- R9 pad 1: +5V -> /Receiver/RX_SHIFT
- R9 pad 2: Net-(Q1-C) -> -15V
- TP1 pad 1: -15V -> +10V
- TP6 pad 1: +5V -> -15V
- TP7 pad 1: +10V -> /TxD
Routing:
- net GND: track 393.8 -> 0.00 mm, vias 1 -> 0
- net -15V: track 239.0 -> 0.00 mm, vias 1 -> 0
- net +10V: track 196.0 -> 0.00 mm, vias 1 -> 0
- net +5V: track 125.5 -> 0.00 mm
- net /TTO_CL: track 85.2 -> 0.00 mm
- net /RDR_EN_CL: track 84.5 -> 0.00 mm
- net /TTI_CL_RET: track 77.0 -> 0.00 mm
- net Net-(D1-K): track 73.1 -> 0.00 mm
- net Net-(D2-K): track 72.8 -> 0.00 mm
- net /TTI_EIA_NEG: track 52.8 -> 0.00 mm
- net /TTI: track 44.2 -> 0.00 mm
- net /RDR_EN: track 43.1 -> 0.00 mm
- net /TTO: track 41.4 -> 0.00 mm
- net /CTS: track 40.9 -> 0.00 mm
- net Net-(D3-K): track 39.4 -> 0.00 mm
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Other:
- board size 125.7 x 62.2 mm -> 125.2 x 61.9 mm
- board text removed: "(c)Scott Finneran 2026 https://github.com/sierrafoxtrot"
- board text removed: "2 3 8 5"
- board text removed: "3 2 5 7"
- board text removed: "3 7 Relay- 4 Relay+ 6"
- board text removed: "3 TTI Return 7 TTO Relay- -15V 4 +10V Relay+ Reader Enable 6 TTO Return"
- board text removed: "ALL LINKS"
- board text removed: "CTS"
- board text removed: "CURRENT LOOP"
- board text removed: "GND"
- board text removed: "PDP-8 Serial AIO (DCE)"
- board text removed: "PDP-8 Serial All-in-One"
- board text removed: "RE"
- board text removed: "RS-232"
- board text removed: "Rev. A"
- board text removed: "Rx"
- board text removed: "Serial Cable"
- board text removed: "Terminal (25 way)"
- board text removed: "Terminal (9 way)"
- board text removed: "Tx"
- board text removed: "W070 Current Loop"

Commit message: Added holeless flip-chip layout. Footprints assigned.
Parts:
- J3: footprint Connector_PCBEdge:DEC_single_short -> Library:DEC_single_short_holeless
- R10, R11, R13, R14, R15, R16, R17, R18, R19, R20, R21, R22, R23, R24, R25, R26, R27, R28, R29, R30, R31, R32, R33, R34, R35, R36, R37, R38, R39, R40, R5, R6, R7, R8, R9: footprint Resistor_THT:R_Axial_DIN0207_L6.3mm_D2.5mm_P10.16mm_Horizontal -> Resistor_THT:R_Axial_DIN0207_L6.3mm_D2.5mm_P7.62mm_Horizontal
- R12, R4: footprint Resistor_THT:R_Axial_DIN0207_L6.3mm_D2.5mm_P10.16mm_Horizontal -> Resistor_THT:R_Axial_DIN0309_L9.0mm_D3.2mm_P12.70mm_Horizontal
- moved R27 268.4 mm to (332.0, 85.0), turned to 0 degrees
- moved R29 244.8 mm to (317.0, 80.0), turned to 0 degrees
- moved Q16 235.3 mm to (301.0, 85.0), turned to 0 degrees
- moved R34 234.5 mm to (324.0, 95.0), turned to 0 degrees
- moved TP13 234.0 mm to (340.0, 75.0), turned to 0 degrees
- moved D10 233.4 mm to (321.0, 62.0), turned to 0 degrees
- moved R28 222.1 mm to (290.0, 80.0), turned to 0 degrees
- moved R31 220.3 mm to (303.0, 54.0), turned to 0 degrees
- moved R38 218.9 mm to (328.0, 75.0), turned to 0 degrees
- moved J5 218.7 mm to (302.0, 74.0), turned to 0 degrees
- moved D14 218.0 mm to (319.0, 66.0), turned to 0 degrees
- moved C11 217.7 mm to (326.0, 85.0), turned to 0 degrees
- moved C10 216.6 mm to (318.0, 95.0), turned to 0 degrees
- moved R33 214.3 mm to (298.0, 100.0), turned to 0 degrees
- moved D12 214.0 mm to (308.0, 65.0), turned to 0 degrees
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
Commit message: New footprints and symbols. PCB layout begun
Parts:
- removed J4, J5: Conn_01x03, Connector_PinHeader_2.54mm:PinHeader_1x03_P2.54mm_Vertical
- removed TP10, TP11, TP12, TP13: TestPoint, TestPoint:TestPoint_Loop_D3.50mm_Drill0.9mm_Beaded
- removed TP7, TP8, TP9: TTI, TestPoint:TestPoint_Loop_D3.50mm_Drill0.9mm_Beaded
- added D16: 1N914, Diode_THT:D_DO-35_SOD27_P7.62mm_Horizontal, F.Cu at (116.1, 143.6)
- added D17: 1N914, Diode_THT:D_DO-35_SOD27_P7.62mm_Horizontal, F.Cu at (118.8, 143.6)
- added D18: 1N914, Diode_THT:D_DO-35_SOD27_P7.62mm_Horizontal, F.Cu at (124.3, 143.6)
- added LK4: Link_01x03, Connector_PinHeader_2.54mm:PinHeader_1x03_P2.54mm_Vertical, F.Cu at (161.3, 126.2)
- added LK5: Link_01x03, Connector_PinHeader_2.54mm:PinHeader_1x03_P2.54mm_Vertical, F.Cu at (161.3, 141.8)
- added R41: 10k, Resistor_THT:R_Axial_DIN0207_L6.3mm_D2.5mm_P7.62mm_Horizontal, F.Cu at (130.5, 143.6)
- added R42: 68, Resistor_THT:R_Axial_DIN0207_L6.3mm_D2.5mm_P7.62mm_Horizontal, F.Cu at (99.9, 135.9)
- added R43: 68, Resistor_THT:R_Axial_DIN0207_L6.3mm_D2.5mm_P7.62mm_Horizontal, F.Cu at (103.1, 143.6)
- D1, D2, D3: value 1N914 -> LED; footprint Diode_THT:D_DO-35_SOD27_P7.62mm_Horizontal -> LED_THT:LED_D3.0mm
- LK1, LK2, LK3: value Conn_01x03 -> Link_01x03
- R1: value 1k -> 27k; footprint Resistor_THT:R_Axial_DIN0414_L11.9mm_D4.5mm_P20.32mm_Horizontal -> Resistor_THT:R_Axial_DIN0207_L6.3mm_D2.5mm_P7.62mm_Horizontal
- R10: value 10k -> 47k
- R11: value 2k7 -> 47k
- R12: value 2k2 -> 47k; footprint Resistor_THT:R_Axial_DIN0309_L9.0mm_D3.2mm_P12.70mm_Horizontal -> Resistor_THT:R_Axial_DIN0207_L6.3mm_D2.5mm_P7.62mm_Horizontal
- R13, R27: value 7k5 -> 10k
- R14: value 47k -> 2k7
- R15: value 100k -> 2k2; footprint Resistor_THT:R_Axial_DIN0207_L6.3mm_D2.5mm_P7.62mm_Horizontal -> Resistor_THT:R_Axial_DIN0309_L9.0mm_D3.2mm_P12.70mm_Horizontal
- R16, R30: value 10k -> 7k5
- R17, R31: value 27k -> 47k
- R18, R32, R8: value 47k -> 100k
- R19, R33: value 100k -> 10k
- R2: value 750R -> 10k; footprint Resistor_THT:R_Axial_DIN0414_L11.9mm_D4.5mm_P20.32mm_Horizontal -> Resistor_THT:R_Axial_DIN0207_L6.3mm_D2.5mm_P7.62mm_Horizontal
- R20, R34: value 33k -> 27k
- R21, R35: value 100k -> 47k
- R22, R24, R36, R38: value 10k -> 100k
- R23, R37: value 10k -> 33k
- R25, R26, R39, R40: value 68 -> 10k
- R28: value 47k -> 68
- R29: value 100k -> 68
- R3: value 750R -> 27k; footprint Resistor_THT:R_Axial_DIN0414_L11.9mm_D4.5mm_P20.32mm_Horizontal -> Resistor_THT:R_Axial_DIN0207_L6.3mm_D2.5mm_P7.62mm_Horizontal
- R4: value 5k1 -> 1k; footprint Resistor_THT:R_Axial_DIN0309_L9.0mm_D3.2mm_P12.70mm_Horizontal -> Resistor_THT:R_Axial_DIN0414_L11.9mm_D4.5mm_P20.32mm_Horizontal
- R5: value 100k -> 750R; footprint Resistor_THT:R_Axial_DIN0207_L6.3mm_D2.5mm_P7.62mm_Horizontal -> Resistor_THT:R_Axial_DIN0414_L11.9mm_D4.5mm_P20.32mm_Horizontal
- R6: value 470k -> 750R; footprint Resistor_THT:R_Axial_DIN0207_L6.3mm_D2.5mm_P7.62mm_Horizontal -> Resistor_THT:R_Axial_DIN0414_L11.9mm_D4.5mm_P20.32mm_Horizontal
- R7: value 47k -> 5k1; footprint Resistor_THT:R_Axial_DIN0207_L6.3mm_D2.5mm_P7.62mm_Horizontal -> Resistor_THT:R_Axial_DIN0309_L9.0mm_D3.2mm_P12.70mm_Horizontal
- R9: value 47k -> 470k
- TP4: value TTO -> TTI
- TP5: value RDR_EN -> TTI
- moved C9 247.1 mm to (88.4, 157.9), turned to 90 degrees
- moved C7 233.5 mm to (97.3, 158.2), turned to 90 degrees
- moved TP6 232.7 mm to (101.1, 109.5), turned to 90 degrees
- moved C11 231.6 mm to (106.5, 158.8)
- moved C5 222.6 mm to (97.8, 104.9), turned to 90 degrees
- moved C3 219.8 mm to (97.8, 94.6), turned to -90 degrees
- moved C10 219.8 mm to (106.5, 154.7)
- moved R29 219.2 mm to (103.1, 128.0), turned to 90 degrees
- moved TP4 217.2 mm to (111.3, 109.5), turned to 90 degrees
- moved D10 215.3 mm to (116.1, 128.0), turned to 90 degrees
- moved D1 214.3 mm to (87.0, 112.7), turned to -90 degrees
- moved D2 208.4 mm to (91.6, 112.7), turned to -90 degrees
- moved R8 207.0 mm to (117.1, 112.3)
- moved R27 206.0 mm to (130.5, 128.0), turned to 90 degrees
- moved R38 203.0 mm to (136.9, 143.6), turned to 90 degrees
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Connections:
- D1 pad 1: GND -> Net-(D1-K)
- D1 pad 2: /TTI_CL -> GND
- D10 pad 1: GND -> /Transmitter/B4
- D11 pad 1: Net-(D11-K) -> /Transmitter/B3
- D11 pad 2: GND -> /Transmitter/Q3_E
- D12 pad 1: Net-(D12-K) -> /Transmitter/Q4_E
- D12 pad 2: /Reader Enable (CTS)/B3 -> /Transmitter/B4
- D13 pad 1: /Reader Enable (CTS)/B4 -> GND
- D14 pad 1: /Reader Enable (CTS)/B3 -> Net-(D14-K)
- D14 pad 2: /Reader Enable (CTS)/Q3_E -> GND
- D15 pad 1: /Reader Enable (CTS)/Q4_E -> Net-(D15-K)
- D15 pad 2: /Reader Enable (CTS)/B4 -> /Reader Enable (CTS)/B3
- D3 pad 1: GND -> -15V
- D4 pad 2: Net-(D4-A) -> /TTI_CL
- D6 pad 1: Net-(D6-K) -> GND
- D6 pad 2: /Transmitter/B3 -> Net-(D6-A)
- D7 pad 1: /Transmitter/B4 -> GND
- D8 pad 1: /Transmitter/B3 -> Net-(D8-K)
- D8 pad 2: /Transmitter/Q3_E -> GND
- D9 pad 1: /Transmitter/Q4_E -> Net-(D9-K)
- D9 pad 2: /Transmitter/B4 -> /Transmitter/B3
- J3 pad AA2: (no net) -> +10V
- J3 pad AB2: (no net) -> -15V
- J3 pad AC2: (no net) -> GND
- J3 pad AD2: (no net) -> /TTI
- J3 pad AE2: (no net) -> unconnected-(J3-Pin_E-PadAE2)
- J3 pad AF2: (no net) -> unconnected-(J3-Pin_F-PadAF2)
- J3 pad AH2: (no net) -> /TTO
- J3 pad AJ2: (no net) -> unconnected-(J3-Pin_J-PadAJ2)
- J3 pad AK2: (no net) -> unconnected-(J3-Pin_K-PadAK2)
- J3 pad AL2: (no net) -> unconnected-(J3-Pin_L-PadAL2)
- J3 pad AM2: (no net) -> /RDR_EN
- J3 pad AN2: (no net) -> unconnected-(J3-Pin_N-PadAN2)
- J3 pad AP2: (no net) -> unconnected-(J3-Pin_P-PadAP2)
- J3 pad AR2: (no net) -> unconnected-(J3-Pin_r-PadAR2)
- J3 pad AS2: (no net) -> unconnected-(J3-Pin_S-PadAS2)
- J3 pad AT2: (no net) -> unconnected-(J3-Pin_T-PadAT2)
- J3 pad AU2: (no net) -> unconnected-(J3-Pin_U-PadAU2)
- J3 pad AV2: (no net) -> unconnected-(J3-Pin_v-PadAV2)
- Q1 pad 2: Net-(D2-K) -> Net-(D5-K)
- Q10 pad 3: Net-(D7-A) -> Net-(D10-A)
- Q11 pad 2: Net-(D10-A) -> Net-(D13-A)
- Q12 pad 2: Net-(D11-K) -> Net-(D14-K)
- Q16 pad 3: Net-(D12-K) -> Net-(D15-K)
- Q17 pad 3: Net-(D13-A) -> Net-(D16-A)
- Q3 pad 2: Net-(D3-A) -> Net-(D6-A)
- Q4 pad 2: Net-(D4-A) -> Net-(D7-A)
- Q5 pad 2: Net-(D5-K) -> Net-(D8-K)
- Q9 pad 3: Net-(D6-K) -> Net-(D9-K)
- R1 pad 1: /TTI_CL_RET -> /TTO
- R1 pad 2: /TTI_CL -> Net-(D1-K)
- R10 pad 1: /Receiver/RX_SHIFT -> /Receiver/RX_SENSE
- R10 pad 2: Net-(D3-A) -> +10V
- R11 pad 1: /TTI_EIA_NEG -> Net-(Q2-B)
- R11 pad 2: GND -> /Receiver/RX_SENSE
- R12 pad 1: /TTI_EIA_NEG -> /Receiver/RX_SHIFT
- R13 pad 1: -15V -> /Receiver/RX_SHIFT
- R13 pad 2: /DEC_TTO_232 -> Net-(D6-A)
- R14 pad 1: /DEC_TTO_232 -> /TTI_EIA_NEG
- R14 pad 2: Net-(D4-A) -> GND
- R15 pad 1: Net-(D4-A) -> /TTI_EIA_NEG
- R15 pad 2: +10V -> -15V
- R16 pad 1: /Transmitter/DEC_IN_INV -> -15V
- R16 pad 2: -15V -> /DEC_TTO_232
- R17 pad 1: Net-(J4-Pin_2) -> /DEC_TTO_232
- R17 pad 2: Net-(D5-K) -> Net-(D7-A)
- R18 pad 1: +10V -> Net-(D7-A)
- R18 pad 2: Net-(D5-K) -> +10V
- R19 pad 1: +10V -> /Transmitter/DEC_IN_INV
- R19 pad 2: /Transmitter/Q1_C -> -15V
- R2 pad 1: -15V -> /TTI
- R2 pad 2: /TTI_CL_RET -> Net-(D2-K)
- R20 pad 1: /Transmitter/Q1_C -> Net-(LK4-Pin_2)
- R20 pad 2: Net-(Q6-B) -> Net-(D8-K)
- R21 pad 2: Net-(Q6-B) -> Net-(D8-K)
- R22 pad 1: /Transmitter/DRV -> +10V
- R22 pad 2: -15V -> /Transmitter/Q1_C
- R23 pad 1: /Transmitter/DRV -> /Transmitter/Q1_C
- R23 pad 2: /Transmitter/B3 -> Net-(Q6-B)
- R24 pad 1: /Transmitter/DRV -> +10V
- R24 pad 2: /Transmitter/B4 -> Net-(Q6-B)
- R25 pad 1: /Transmitter/Q3_E -> /Transmitter/DRV
- R25 pad 2: /RxD -> -15V
- R26 pad 1: /RxD -> /Transmitter/DRV
- R26 pad 2: /Transmitter/Q4_E -> /Transmitter/B3
- R27 pad 1: -15V -> /Transmitter/DRV
- R27 pad 2: /DEC_REN_232 -> /Transmitter/B4
- R28 pad 1: /DEC_REN_232 -> /Transmitter/Q3_E
- R28 pad 2: Net-(D10-A) -> /RxD
- R29 pad 1: Net-(D10-A) -> /RxD
- R29 pad 2: +10V -> /Transmitter/Q4_E
- R3 pad 1: /TTO_CL_RET -> /RDR_EN
- R3 pad 2: -15V -> Net-(D3-A)
- R30 pad 1: /Reader Enable (CTS)/DEC_IN_INV -> -15V
- R30 pad 2: -15V -> /DEC_REN_232
- R31 pad 1: Net-(J5-Pin_2) -> /DEC_REN_232
- R31 pad 2: Net-(D11-K) -> Net-(D13-A)
- R32 pad 1: +10V -> Net-(D13-A)
- R32 pad 2: Net-(D11-K) -> +10V
- R33 pad 1: +10V -> /Reader Enable (CTS)/DEC_IN_INV
- R33 pad 2: /Reader Enable (CTS)/Q1_C -> -15V
- R34 pad 1: /Reader Enable (CTS)/Q1_C -> Net-(LK5-Pin_2)
- R34 pad 2: Net-(Q13-B) -> Net-(D14-K)
- R35 pad 2: Net-(Q13-B) -> Net-(D14-K)
- R36 pad 1: /Reader Enable (CTS)/DRV -> +10V
- R36 pad 2: -15V -> /Reader Enable (CTS)/Q1_C
- R37 pad 1: /Reader Enable (CTS)/DRV -> /Reader Enable (CTS)/Q1_C
- R37 pad 2: /Reader Enable (CTS)/B3 -> Net-(Q13-B)
- R38 pad 1: /Reader Enable (CTS)/DRV -> +10V
- R38 pad 2: /Reader Enable (CTS)/B4 -> Net-(Q13-B)
- R39 pad 1: /Reader Enable (CTS)/Q3_E -> /Reader Enable (CTS)/DRV
- R39 pad 2: /CTS -> -15V
- R4 pad 1: GND -> /TTI_CL_RET
- R4 pad 2: /TxD -> /TTI_CL
- R40 pad 1: /CTS -> /Reader Enable (CTS)/DRV
- R40 pad 2: /Reader Enable (CTS)/Q4_E -> /Reader Enable (CTS)/B3
- R5 pad 1: /TxD -> -15V
- R5 pad 2: Net-(D2-K) -> /TTI_CL_RET
- R6 pad 1: GND -> /TTO_CL_RET
- R6 pad 2: Net-(D2-K) -> -15V
- R7 pad 1: /Receiver/RX_SENSE -> GND
- R7 pad 2: +10V -> /TxD
- R8 pad 1: Net-(Q2-B) -> /TxD
- R8 pad 2: /Receiver/RX_SENSE -> Net-(D5-K)
- R9 pad 1: /Receiver/RX_SHIFT -> GND
- R9 pad 2: -15V -> Net-(D5-K)
- TP3 pad 1: /TTI -> -15V
- TP4 pad 1: /TTO -> /TxD
- TP5 pad 1: /RDR_EN -> /RxD
- TP6 pad 1: -15V -> /CTS
Routing:
- net GND: track 0.00 -> 375.0 mm
- net +10V: track 0.00 -> 369.5 mm
- net -15V: track 0.00 -> 362.6 mm
- net Net-(D2-K): track 0.00 -> 96.5 mm
- net /TTO_CL: track 0.00 -> 91.2 mm
- net Net-(D1-K): track 0.00 -> 91.1 mm
- net /RDR_EN_CL: track 0.00 -> 88.5 mm
- net Net-(D3-A): track 0.00 -> 78.5 mm
- net /TTO_CL_RET: track 0.00 -> 63.3 mm
- net /CTS: track 0.00 -> 62.4 mm
- net /TTI_CL_RET: track 0.00 -> 58.6 mm
- net /TxD: track 0.00 -> 56.0 mm
- net /DEC_REN_232: track 0.00 -> 52.6 mm
- net /RxD: track 0.00 -> 35.6 mm
- net /DEC_TTO_232: track 0.00 -> 35.0 mm
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
Commit message: ERC & DRC clear. Layout complete
Parts:
- TP1: value TTI -> +10V
- TP2: value TTI -> GND
- TP3: value TTI -> -15V
- TP4: value TTI -> TxD
- TP5: value TTI -> RxD
- TP6: value TTI -> CTS
- moved C7 79.7 mm to (156.7, 105.2), turned to 180 degrees
- moved C6 68.5 mm to (136.6, 105.2), turned to 180 degrees
- moved TP2 48.8 mm to (165.6, 142.7)
- moved C9 47.4 mm to (113.3, 117.6), turned to 180 degrees
- moved TP1 43.3 mm to (165.6, 131.3)
- moved C8 37.0 mm to (110.8, 132.1), turned to 0 degrees
- moved TP3 36.2 mm to (165.6, 127.0)
- moved C11 26.7 mm to (105.2, 132.1)
- moved C10 9.04 mm to (103.1, 146.3), turned to 180 degrees
- moved R2 1.52 mm to (185.7, 104.6)
- moved C1 1.05 mm to (187.1, 91.1)
- moved C2 1.05 mm to (183.9, 96.1)
- moved D6 0.51 mm to (159.5, 112.8)
- moved J2 0.25 mm to (95.4, 127.0)
- moved Q3 0.25 mm to (163.6, 112.4)
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Routing:
- net GND: track 375.0 -> 416.0 mm
- net +10V: track 369.5 -> 388.0 mm
- net -15V: track 362.6 -> 378.4 mm
- net /TxD: track 56.0 -> 48.0 mm
- net Net-(D2-K): track 96.5 -> 98.1 mm
- net Net-(D6-A): track 16.2 -> 17.6 mm
- net /RDR_EN_CL: track 88.5 -> 89.6 mm
Other:
- board text added: "(c)Scott Finneran 2026 https://github.com/sierrafoxtrot"
- board text added: "2 3 8 5"
- board text added: "3 2 5 7"
- board text added: "3 7 Relay- 4 Relay+ 6"
- board text added: "3 TTI Return 7 TTO Relay- -15V 4 +10V Relay+ Reader En. 6 TTO Return"
- board text added: "ALL LINKS"
- board text added: "CTS"
- board text added: "CURRENT LOOP"
- board text added: "GND"
- board text added: "PDP-8 Serial AIO (DCE)"
- board text added: "PDP-8 Serial All-in-One"
- board text added: "REN"
- board text added: "RS-232"
- board text added: "RS-232 DCE"
- board text added: "Rx"
- board text added: "Serial Cable"
- board text added: "Serial Cable Wiring Diagram"
- board text added: "TELETYPE CONNECTOR W070-PLUS-A"
- board text added: "TTI"
- board text added: "TTO"
- board text added: "Terminal (25 way)"
- board text added: "Terminal (9 way)"
- board text added: "Tx"
- board text added: "W070 Current Loop"

Commit message: PCB cleanup
Routing:
- net +10V: track 388.0 -> 387.4 mm
Changed lines of the file:
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@@
 	)
 	(segment
-		(start 108.966 130.302)
-		(end 106.974 130.302)
+		(start 106.974 130.302)
+		(end 111.486 130.302)
 		(width 0.508)
 		(layer "B.Cu")
@@
 	)
 	(segment
-		(start 181.292501 126.555499)
-		(end 182.753 128.015999)
-		(width 0.508)
-		(layer "B.Cu")
-		(net 1)
-	)
-	(segment
 		(start 159.004 112.776)
 		(end 157.48 114.3)
@@
 	)
 	(segment
-		(start 181.267704 142.101005)
+		(start 179.934205 140.767506)
 		(end 182.728203 143.561505)
 		(width 0.508)
@@
 	)
 	(segment
-		(start 179.934205 140.767506)
-		(end 181.267704 142.101005)
-		(width 0.508)
-		(layer "B.Cu")
-		(net 1)
-	)
-	(segment
 		(start 140.462 132.08)
 		(end 113.264 132.08)
@@
 	)
 	(segment
-		(start 111.486 130.302)
-		(end 108.966 130.302)
-		(width 0.508)
-		(layer "B.Cu")
-		(net 1)
-	)
-	(segment
 		(start 163.322 112.268)
 		(end 161.29 112.268)
@@
 	(segment
 		(start 179.959002 125.222)
-		(end 181.292501 126.555499)
+		(end 182.753 128.015999)
 		(width 0.508)
 		(layer "B.Cu")
@@
 	)
 	(segment
-		(start 110.744 145.288)
+		(start 110.744 145.796)
 		(end 110.744 143.403274)
 		(width 0.508)
@@
 	(segment
 		(start 134.111999 146.304)
-		(end 134.365999 146.05)
+		(end 136.906 143.509999)
 		(width 0.508)
 		(layer "F.Cu")
@@
 	)
 	(segment
-		(start 110.744 145.796)
-		(end 110.744 145.288)
-		(width 0.508)
-		(layer "F.Cu")
-		(net 2)
-	)
-	(segment
 		(start 134.365999 130.556)
 		(end 111.506 130.556)
@@
 	)
 	(segment
-		(start 136.906 143.509999)
-		(end 134.365999 146.05)
-		(width 0.508)
-		(layer "F.Cu")
-		(net 2)
-	)
-	(segment
 		(start 110.744 127.909274)
 		(end 112.161275 126.491999)
@@
 	)
 	(segment
-		(start 154.559 128.015999)
-		(end 154.559 128.143)
-		(width 0.508)
-		(layer "B.Cu")
-		(net 2)
-	)
-	(segment
 		(start 142.494 102.362)
 		(end 144.272 104.14)
@@
 	)
 	(segment
-		(start 201.922 91.353)
-		(end 202.2 91.075)
-		(width 0.508)
-		(layer "B.Cu")
-		(net 2)
-	)
-	(segment
-		(start 154.534203 143.561505)
-		(end 154.534203 143.688506)
-		(width 0.508)
-		(layer "B.Cu")
-		(net 2)
-	)
-	(segment
 		(start 144.123999 129.54)
 		(end 138.430001 129.54)
@@
 	)
 	(segment
-		(start 188.976 143.028709)
-		(end 186.157203 145.847506)
-		(width 0.508)
-		(layer "F.Cu")
-		(net 3)
-	)
-	(segment
-		(start 190.246 141.758709)
-		(end 188.976 143.028709)
+		(start 186.157203 145.847506)
+		(end 190.246 141.758709)
 		(width 0.508)
 		(layer "F.Cu")
@@
 	)
 	(segment
-		(start 170.18 100.33)
-		(end 170.434 100.076)
-		(width 0.508)
-		(layer "B.Cu")
-		(net 3)
-	)
-	(segment
 		(start 187.047 94.25)
 		(end 202.2 94.25)
@@
 	)
 	(segment
-		(start 124.46 120.395999)
-		(end 124.46 120.65)
-		(width 0.3048)
-		(layer "F.Cu")
-		(net 12)
-	)
-	(segment
 		(start 116.078 124.421199)
 		(end 113.7038 122.046999)
@@
 	)
 	(segment
-		(start 124.435203 135.941505)
-		(end 124.435203 136.195506)
-		(width 0.3048)
-		(layer "F.Cu")
-		(net 18)
-	)
-	(segment
 		(start 113.679003 137.592505)
 		(end 112.624203 137.592505)
@@
 	(segment
 		(start 105.893203 143.307506)
-		(end 105.893204 143.307505)
+		(end 107.544203 143.307505)
 		(width 0.3048)
 		(layer "B.Cu")
@@
 	)
 	(segment
-		(start 105.893204 143.307505)
-		(end 107.544203 143.307505)
-		(width 0.3048)
-		(layer "B.Cu")
-		(net 20)
-	)
-	(segment
 		(start 110.719202 144.577505)
 		(end 109.449203 143.307506)
@@
 	)
 	(segment
-		(start 114.3 108.966)
+		(start 114.3 109.474)
 		(end 114.3 105.41)
 		(width 0.3048)
@@
 		(width 0.3048)
 		(layer "F.Cu")
-		(net 23)
-	)
-	(segment
-		(start 114.3 109.474)
-		(end 114.3 108.966)
-		(width 0.3048)
-		(layer "F.Cu")

Commit message: Geographic reannotation of PCB
Parts:
- moved R2 20.3 mm to (142.9, 95.2), turned to 0 degrees
- moved R16 7.62 mm to (100.0, 128.0), turned to 90 degrees
- moved R26 7.62 mm to (169.7, 128.0), turned to 90 degrees
- moved R28 7.62 mm to (179.8, 128.0), turned to 90 degrees
- moved R29 7.62 mm to (176.4, 128.0), turned to 90 degrees
- moved R15 7.62 mm to (185.7, 112.3), turned to 90 degrees
- moved R31 7.62 mm to (99.9, 143.6), turned to 90 degrees
- moved R7 7.62 mm to (140.7, 112.8), turned to 90 degrees
- moved R41 7.57 mm to (169.6, 143.5), turned to 90 degrees
- moved R42 7.57 mm to (176.4, 143.5), turned to 90 degrees
- moved R43 7.57 mm to (179.8, 143.5), turned to 90 degrees
- moved C4 5.00 mm to (183.9, 91.1), turned to -90 degrees
- renumbered C4 to C1, C11 to C10, C10 to C11, C3 to C2, C5 to C3, C2 to C4, C1 to C5, C9 to C8, C8 to C9, D12 to D10, D8 to D11, D7 to D12, D16 to D13, D17 to D14, D18 to D16, D14 to D17, D13 to D18, D5 to D4, D4 to D5, D10 to D7, D9 to D8, D11 to D9, Q4 to Q10, Q17 to Q11, Q15 to Q12, Q16 to Q13, Q12 to Q15, Q13 to Q16, Q11 to Q17, Q10 to Q4, Q8 to Q5, Q9 to Q6, Q5 to Q8, Q6 to Q9, R4 to R1, R13 to R10, R14 to R11, R15 to R12, R1 to R13, R3 to R14, R2 to R15, R28 to R16, R29 to R17, R26 to R18, R25 to R19, R5 to R2, R27 to R20, R24 to R21, R23 to R22, R22 to R23, R21 to R24, R20 to R25, R17 to R26, R16 to R27, R18 to R28, R19 to R29, R6 to R3, R43 to R30, R42 to R31, R40 to R32, R39 to R33, R41 to R34, R37 to R35, R38 to R36, R36 to R37, R35 to R38, R34 to R39, R7 to R4, R30 to R40, R31 to R41, R33 to R42, R32 to R43, R9 to R5, R8 to R6, R11 to R7, R10 to R8, R12 to R9, TP6 to TP1, TP5 to TP2, TP4 to TP3, TP3 to TP4, TP1 to TP5, TP2 to TP6
Connections:
- C4 pad 1: GND -> -15V
- C4 pad 2: -15V -> GND
- D12 pad 2: Net-(D7-A) (its old number) -> Net-(D12-A)
- D18 pad 2: Net-(D13-A) (its old number) -> Net-(D18-A)
- Q10 pad 2: Net-(D7-A) (its old number) -> Net-(D12-A)
- Q17 pad 2: Net-(D13-A) (its old number) -> Net-(D18-A)
- R15 pad 1: /TTI -> Net-(D2-K)
- R15 pad 2: Net-(D2-K) -> /TTI
- R16 pad 1: /Transmitter/Q3_E -> /RxD
- R16 pad 2: /RxD -> /Transmitter/Q3_E
- R2 pad 1: -15V -> /TTI_CL_RET
- R2 pad 2: /TTI_CL_RET -> -15V
- R26 pad 1: /DEC_TTO_232 -> Net-(D12-A)
- R26 pad 2: Net-(D7-A) (its old number) -> /DEC_TTO_232
- R28 pad 1: Net-(D7-A) (its old number) -> +10V
- R28 pad 2: +10V -> Net-(D12-A)
- R29 pad 1: /Transmitter/DEC_IN_INV -> -15V
- R29 pad 2: -15V -> /Transmitter/DEC_IN_INV
- R31 pad 1: /Reader Enable (CTS)/Q3_E -> /CTS
- R31 pad 2: /CTS -> /Reader Enable (CTS)/Q3_E
- R41 pad 1: /DEC_REN_232 -> Net-(D18-A)
- R41 pad 2: Net-(D13-A) (its old number) -> /DEC_REN_232
- R42 pad 1: /Reader Enable (CTS)/DEC_IN_INV -> -15V
- R42 pad 2: -15V -> /Reader Enable (CTS)/DEC_IN_INV
- R43 pad 1: Net-(D13-A) (its old number) -> +10V
- R43 pad 2: +10V -> Net-(D18-A)
- R7 pad 1: Net-(Q2-B) -> /Receiver/RX_SENSE
- R7 pad 2: /Receiver/RX_SENSE -> Net-(Q2-B)
Routing:
- net Net-(D18-A): track 0.00 -> 26.7 mm
- net Net-(D13-A) (its old number): track 26.7 -> 0.00 mm
- net Net-(D7-A) (its old number): track 26.7 -> 0.00 mm
- net Net-(D12-A): track 0.00 -> 26.7 mm

Commit message: Updated copyright symbol
Other:
- board text added: "©Scott Finneran 2026 https://github.com/sierrafoxtrot"
- board text removed: "(c)Scott Finneran 2026 https://github.com/sierrafoxtrot"
- board text removed: "Serial Cable"
